File: PCB/FluxEngine_Hat_CDC_9406_cfg_2.kicad_pcb (KiCad board)
At the start: 2 copper layers, 83.3 x 24.1 mm, 3 parts, among them J1 CY8CKIT-059, P1 FDD_IBMPC_host, P2 CDC_9406_type_2

Commit message: readme
Other:
- board text added: "3.5 inch 5.25 inch"
- board text added: "8 inch CDC 9406 cfg 2"
- board text removed: "CDC9406-p2"
Changed lines of the file:
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@@
 		)
 	)
-	(gr_text "CDC9406-p2"
-		(at 103.805001 106.959999 0)
+	(gr_text "8 inch\nCDC 9406\ncfg 2"
+		(at 107.315001 95.249999 0)
 		(layer "F.SilkS")
 		(effects
@@
 				(bold yes)
 			)
-			(justify left)
+			(justify bottom)
 		)
 	)
+	(gr_text "3.5 inch\n5.25 inch"
+		(at 121.920001 92.074999 90)
+		(layer "F.SilkS")
+		(effects
+			(font
+				(size 1.016 1.016)
+				(thickness 0.2032)
+				(bold yes)
+			)
+			(justify bottom)
+		)
+	)
