File: PCB/FluxEngine_Hat_CDC.kicad_sch (KiCad schematic)
At the start: 3 parts, among them J1 CY8CKIT-059, P1 FDC_BUS_IBMPC, P2 FDC_BUS_CDC

Commit message: readme & remove slash from page names
Other:
- title: FluxEngine_Hat for PC and CDC/MPI -> FluxEngine_Hat for PC and CDC
Changed lines of the file:
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@@
 	(paper "User" 298.45 217.322)
 	(title_block
-		(title "FluxEngine_Hat for PC and CDC/MPI")
+		(title "FluxEngine_Hat for PC and CDC")
 		(date "2024-04-25")
 		(rev "002")
