File: PCB/FluxEngine_Hat_CDC_ALT1.kicad_pcb (KiCad board)
At the start: 2 copper layers, 83.3 x 24.1 mm, 5 parts, among them J1 CY8CKIT-059, J2 5V, J3 24V, P1 FDC_BUS_IBMPC, P2 FDC_BUS_CDC_alt1

Commit message: readme & remove slash from page names
Other:
- board text added: "50pin: CDC/MPI {dblquote}ALT1{dblquote} ex: 77618003"
- board text removed: "50pin: CDC/MPI alt1 ex: 77618003"
