File: PCB/FluxEngine_Hat_CDC_ALT1.kicad_sch (KiCad schematic)
At the start: 5 parts, among them J1 CY8CKIT-059, J2 5V, J3 24V, P1 FDC_BUS_IBMPC, P2 FDC_BUS_CDC_alt1

Commit message: readme & remove slash from page names
Other:
- title: FluxEngine_Hat for PC and CDC/MPI alt1 -> FluxEngine_Hat for PC and CDC ALT1
Changed lines of the file:
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@@
 	(paper "User" 298.45 217.322)
 	(title_block
-		(title "FluxEngine_Hat for PC and CDC/MPI alt1")
+		(title "FluxEngine_Hat for PC and CDC ALT1")
 		(date "2024-04-25")
 		(rev "002")
@@
 		)
 		(instances
-			(project "FluxEngine_Hat_CDC_alt1"
+			(project "FluxEngine_Hat_CDC_ALT1"
 				(path "/72d4cbf5-bf28-4978-b5d4-f13155888c6e"
 					(reference "J2")
@@
 		)
 		(instances
-			(project "FluxEngine_Hat_CDC_alt1"
+			(project "FluxEngine_Hat_CDC_ALT1"
 				(path "/72d4cbf5-bf28-4978-b5d4-f13155888c6e"
 					(reference "#PWR01")
@@
 		)
 		(instances
-			(project "FluxEngine_Hat_CDC_alt1"
+			(project "FluxEngine_Hat_CDC_ALT1"
 				(path "/72d4cbf5-bf28-4978-b5d4-f13155888c6e"
 					(reference "J3")
@@
 		)
 		(instances
-			(project "FluxEngine_Hat_CDC_alt1"
+			(project "FluxEngine_Hat_CDC_ALT1"
 				(path "/72d4cbf5-bf28-4978-b5d4-f13155888c6e"
 					(reference "#PWR03")
@@
 		)
 		(instances
-			(project "FluxEngine_Hat_CDC_alt1"
+			(project "FluxEngine_Hat_CDC_ALT1"
 				(path "/72d4cbf5-bf28-4978-b5d4-f13155888c6e"
 					(reference "#PWR06")
@@
 		)
 		(instances
-			(project "FluxEngine_Hat_CDC_alt1"
+			(project "FluxEngine_Hat_CDC_ALT1"
 				(path "/72d4cbf5-bf28-4978-b5d4-f13155888c6e"
 					(reference "J1")
@@
 		)
 		(instances
-			(project "FluxEngine_Hat_CDC_alt1"
+			(project "FluxEngine_Hat_CDC_ALT1"
 				(path "/72d4cbf5-bf28-4978-b5d4-f13155888c6e"
 					(reference "P2")
@@
 		)
 		(instances
-			(project "FluxEngine_Hat_CDC_alt1"
+			(project "FluxEngine_Hat_CDC_ALT1"
 				(path "/72d4cbf5-bf28-4978-b5d4-f13155888c6e"
 					(reference "#PWR08")
@@
 		)
 		(instances
-			(project "FluxEngine_Hat_CDC_alt1"
+			(project "FluxEngine_Hat_CDC_ALT1"
 				(path "/72d4cbf5-bf28-4978-b5d4-f13155888c6e"
 					(reference "P1")
@@
 		)
 		(instances
-			(project "FluxEngine_Hat_CDC_alt1"
+			(project "FluxEngine_Hat_CDC_ALT1"
 				(path "/72d4cbf5-bf28-4978-b5d4-f13155888c6e"
 					(reference "#PWR07")
@@
 		)
 		(instances
-			(project "FluxEngine_Hat_CDC_alt1"
+			(project "FluxEngine_Hat_CDC_ALT1"
 				(path "/72d4cbf5-bf28-4978-b5d4-f13155888c6e"
 					(reference "#PWR02")
@@
 		)
 		(instances
-			(project "FluxEngine_Hat_CDC_alt1"
+			(project "FluxEngine_Hat_CDC_ALT1"
 				(path "/72d4cbf5-bf28-4978-b5d4-f13155888c6e"
 					(reference "#PWR04")
