File: PCB/FluxEngine_Hat_CDC_9406_STD.kicad_sch (KiCad schematic)
At the start: 5 parts, among them J1 CY8CKIT-059, J2 5V, J3 24V, P1 FDC_BUS_IBMPC, P2 FDC_BUS_CDC_alt1

Commit message: more CDC work
Parts:
- removed J2: 5V, 000_LOCAL:ScrewTerminal_1x02_P3.5mm_vertical, symbol 000_LOCAL:Screw_Terminal_01x02
- removed J3: 24V, 000_LOCAL:ScrewTerminal_1x02_P3.5mm_vertical, symbol 000_LOCAL:Screw_Terminal_01x02
- removed P2: FDC_BUS_CDC_alt1, 000_LOCAL:IDC-Header_2x25_P2.54mm_Latch_Vertical, symbol 000_LOCAL:FDC_BUS_CDC_alt1
- added J2: Screw_Terminal_01x04, 000_LOCAL:ScrewTerminal_1x04_P3.5mm_vertical, symbol 000_LOCAL:Screw_Terminal_01x04
- added P2: FDC_BUS_CDC_9406_STD, 000_LOCAL:IDC-Header_2x25_P2.54mm_Latch_Vertical, symbol 000_LOCAL:FDC_BUS_CDC_9406_STD
Connections:
- net 24VDC: now also J2.1 (Pin_1), P2.18 (24VDC), P2.20 (24VDC), P2.22 (24VDC)
- net 5VDC: now also J2.3 (Pin_3), P2.2 (5VDC), P2.4 (5VDC), P2.6 (5VDC)
- net DIR: now also P2.38 (DIR)
- net GND: now also J2.2 (Pin_2), J2.4 (Pin_4), P2.1 (GND), P2.11 (GND), P2.13 (GND), P2.15 (GND), P2.17 (24VGND), P2.19 (24VGND), P2.21 (24VGND), P2.23 (GND), P2.25 (GND), P2.27 (GND), P2.29 (GND), P2.3 (GND), P2.31 (GND), P2.33 (GND), P2.35 (GND), P2.37 (GND), P2.39 (GND), P2.41 (GND), P2.43 (GND), P2.45 (GND), P2.47 (GND), P2.49 (GND), P2.5 (GND), P2.7 (GND), P2.9 (GND)
- net SIDE: now also P2.32 (SIDE)
- net ~{DSKCHG}: now also P2.12 (~{RDY})
- net ~{INDEX}: now also P2.28 (~{INDEX})
- net ~{MOTB}: now also P2.26 (~{HLD})
- net ~{RDATA}: now also P2.34 (~{RDATA})
- net ~{STEP}: now also P2.46 (~{STEP})
- net ~{TG43}: now also P2.44 (~{TG43})
- net ~{TRK0}: now also P2.30 (~{TRK0})
- net ~{WDATA}: now also P2.42 (~{WDATA})
- net ~{WGATE}: now also P2.40 (~{WREN})
- net ~{WPROT}: now also P2.24 (~{WPROT})
Other:
- note added: "For later Control Data / Magnetic Peripherals drives with DC power on the I/O cable and STEP+DIRECTION NOT for Shugart-compatible or most other 8-inch drives."
- note removed: "Special for SOME Control Data / Magnetic Peripherals drives with DC power on the IO cable. NOT for most CDC/MPI models. NOT for Shugart SA800-851 or most other 8-inch drives."
- title: FluxEngine_Hat for PC and CDC ALT1 -> FluxEngine_Hat for PC and CDC 9406-std
