File: PCB/FluxEngine_Hat_CDC_DaisyChain.kicad_pcb (KiCad board)
At the start: 2 copper layers, 83.3 x 24.1 mm, 3 parts, among them J1 CY8CKIT-059, P1 FDC_BUS_IBMPC, P2 FDC_BUS_CDC

Commit message: more CDC work
Parts:
- P2: value FDC_BUS_CDC -> FDC_BUS_CDC_DaisyChain
Other:
- board text added: "34-pin: IBMPC"
- board text added: "50-pin: CDC {dblquote}daisy chain{dblquote} ex: 77618019"
- board text added: "8 inch CDC daisy chain"
- board text removed: "34pin: IBMPC"
- board text removed: "50pin: Most CDC/MPI models (NOT Shugart)"
- board text removed: "8 inch CDC/MPI (NOT Shugart)"
