File: PCB/FluxEngine_Hat_CDC_DaisyChain.kicad_sch (KiCad schematic)
At the start: 3 parts, among them J1 CY8CKIT-059, P1 FDC_BUS_IBMPC, P2 FDC_BUS_CDC

Commit message: more CDC work
Parts:
- removed P2: FDC_BUS_CDC, 000_LOCAL:IDC-Header_2x25_P2.54mm_Latch_Vertical, symbol 000_LOCAL:FDC_BUS_CDC
- added P2: FDC_BUS_CDC_DaisyChain, 000_LOCAL:IDC-Header_2x25_P2.54mm_Latch_Vertical, symbol 000_LOCAL:FDC_BUS_CDC_DaisyChain
Connections:
- net DIR: now also P2.14 (DIR)
- net GND: now also P2.1 (GND), P2.11 (GND), P2.13 (GND), P2.15 (GND), P2.17 (GND), P2.19 (GND), P2.21 (GND), P2.23 (GND), P2.25 (GND), P2.27 (GND), P2.29 (GND), P2.3 (GND), P2.31 (GND), P2.33 (GND), P2.35 (GND), P2.37 (GND), P2.39 (GND), P2.41 (GND), P2.43 (GND), P2.45 (GND), P2.47 (GND), P2.49 (GND), P2.5 (GND), P2.7 (GND), P2.9 (GND)
- net SIDE: now also P2.40 (SIDE)
- net ~{DSB}: now also P2.20 (~{DS1})
- net ~{DSKCHG}: now also P2.28 (~{RDY1})
- net ~{INDEX}: now also P2.8 (~{INDEX})
- net ~{MOTB}: now also P2.4 (~{HLD})
- net ~{RDATA}: now also P2.2 (~{RDATA})
- net ~{STEP}: now also P2.12 (~{STEP})
- net ~{TG43}: now also P2.10 (~{TG43})
- net ~{TRK0}: now also P2.6 (~{TRK0})
- net ~{WDATA}: now also P2.18 (~{WDATA})
- net ~{WGATE}: now also P2.16 (~{WREN})
- net ~{WPROT}: now also P2.36 (~{WPROT})
Other:
- note added: "For Control Data / Magnetic Peripherals drives with "Daisy Chain" interface. NOT for Shugart-compatible or most other 8-inch drives."
- note removed: "Supports most Control Data / Magnetic Peripherals drives. NOT for Shugart SA800-851 or most other 8-inch drives!"
- title: FluxEngine_Hat for PC and CDC -> FluxEngine_Hat for PC and CDC DaisyChain
