File: PCB/FluxEngine_Hat_CDC-standard.kicad_pcb (KiCad board)
At the start: 2 copper layers, 83.3 x 24.1 mm, 7 parts, among them J1 CY8CKIT-059, J2 Screw_Terminal_01x04, P1 FDC_BUS_IBMPC, P2 FDC_BUS_CDC_9406_STD, U1 74HC00

Commit message: silkscreen, pics
Routing:
- net /DIRECTION: track 71.9 -> 72.5 mm
- net /~{STEP}: track 71.1 -> 71.6 mm
- net GND: vias 51 -> 45

Commit message: fix CDC-standard backwards step_in/step_out decoding
Parts:
- added JP2: Jumper_3_Bridged12, 000_LOCAL:PinHeader_1x03_P2.54mm_Vertical, B.Cu at (105.2, 103.0)
- JP1: value Jumper_3_Bridged12_x_2 -> Jumper_3_Bridged12; footprint 000_LOCAL:PinHeader_2x03_P2.54mm_Vertical -> 000_LOCAL:PinHeader_1x03_P2.54mm_Vertical
- U1: value 74HC00 -> LVC1G19; footprint 000_LOCAL:TSSOP-14_4.4x5mm_P0.65mm -> 000_LOCAL:SOT-363_SC-70-6
- moved C1 4.95 mm to (106.4, 100.5), turned to 180 degrees
- moved JP1 2.54 mm to (105.2, 106.0)
- moved U1 1.48 mm to (107.1, 97.7), turned to -90 degrees
Connections:
- JP1 pad 1: /DIRECTION -> /~{STEP}
- JP1 pad 2: /~{STEP} -> /~{STEP}/~{STEP_OUT}
- JP1 pad 3: /DIR/~{STEP_IN} -> /~{STEP_OUT}
- U1 pad 1: /~{STEP} -> /DIRECTION
- U1 pad 2: /~{STEP} -> GND
- U1 pad 3: Net-(U1-Pad10) -> /~{STEP}
- U1 pad 4: /DIRECTION -> /~{STEP_IN}
- U1 pad 5: /DIRECTION -> VCC
- U1 pad 6: Net-(U1-Pad6) -> /~{STEP_OUT}
Routing:
- net Net-(U1-Pad10): track 8.77 -> 0.00 mm
- net /DIRECTION: track 72.5 -> 63.8 mm
- net Net-(U1-Pad6): track 5.72 -> 0.00 mm
- net VCC: track 11.1 -> 14.6 mm
- net /~{STEP}: track 71.6 -> 68.4 mm
- net /~{STEP_IN}: track 7.57 -> 5.41 mm
- net /~{STEP_OUT}: track 11.5 -> 9.76 mm, vias 1 -> 0
- net /DIR/~{STEP_IN}: track 55.7 -> 55.1 mm
- net GND: vias 45 -> 36
Other:
- board text added: "DIR"
- board text added: "STEP"
- board text added: "STEP_IN"
- board text added: "STEP_OUT"
- board text removed: "OLD NEW"
