File: PCB/FluxEngine_Hat_Shugart.kicad_sch (KiCad schematic)
At the start: 6 parts, among them J1 CY8CKIT-059, P1 FDC_BUS_IBMPC, P2 FDC_BUS_SA851

Commit message: staggered rows offset & direction
Other:
- title: FluxEngine_Hat for PC and Shugart -> FluxEngine_Hat_Shugart
Changed lines of the file:
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@@
 	(paper "User" 298.45 217.322)
 	(title_block
-		(title "FluxEngine_Hat for PC and Shugart")
-		(date "2024-05-27")
+		(title "FluxEngine_Hat_Shugart")
+		(date "2024-08-08")
 		(rev "015")
 		(company "Brian K. White - b.kenyon.w@gmail.com")
