File: PCB/FluxEngine_Hat_Shugart.kicad_pcb (KiCad board)
At the start: 2 copper layers, 83.3 x 24.1 mm, 6 parts, among them J1 CY8CKIT-059, P1 FDC_BUS_IBMPC, P2 FDC_BUS_SA851

Commit message: shugart silkscreen
Other:
- board text added: "CY8CKIT-059 this side face up"
- board text removed: "CY8CKIT-059 usb & button face away from hat"
Changed lines of the file:
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@@
 		)
 	)
-	(gr_text "CY8CKIT-059  usb & button face away from hat"
+	(gr_text "CY8CKIT-059 this side face up"
 		(at 147.955001 104.139999 0)
 		(layer "B.SilkS")
